Commit message: Modification to work online

File: hsky_sensor_frame_description/urdf/hsky_sensor.urdf (robot description, URDF)
Before this commit: robot husky, 21 links, 20 joints
Links:
- link base_link: geometry collision box size=0.7899200000000001 0.5709 0.10375; collision box size=0.9874 0.5709 0.12375
- link front_bumper_link: geometry visual mesh filename=../meshes/bumper.dae
- link front_laser: geometry collision mesh filename=../meshes/ust-10lx.stl scale=1 1 1; visual mesh filename=../meshes/ust-10lx.dae scale=1 1 1
- link front_left_wheel_link: geometry collision cylinder length=0.1143 radius=0.1651; visual mesh filename=../meshes/wheel.dae
- link front_mount: geometry collision mesh filename=../meshes/front_laser_mount.stl scale=0.001 0.001 0.001; visual mesh filename=../meshes/front_laser_mount.dae scale=0.001 0.001 0.001
- link front_right_wheel_link: geometry collision cylinder length=0.1143 radius=0.1651; visual mesh filename=../meshes/wheel.dae
- link os_sensor: geometry collision mesh filename=../meshes/os1_64.stl; visual mesh filename=../meshes/os1_64.dae
- link rear_bumper_link: geometry visual mesh filename=../meshes/bumper.dae
- link rear_laser: geometry collision mesh filename=../meshes/ust-10lx.stl scale=1 1 1; visual mesh filename=../meshes/ust-10lx.dae scale=1 1 1
- link rear_left_wheel_link: geometry collision cylinder length=0.1143 radius=0.1651; visual mesh filename=../meshes/wheel.dae
- link rear_mount: geometry collision mesh filename=../meshes/front_laser_mount.stl scale=0.001 0.001 0.001; visual mesh filename=../meshes/front_laser_mount.dae scale=0.001 0.001 0.001
- link rear_right_wheel_link: geometry collision cylinder length=0.1143 radius=0.1651; visual mesh filename=../meshes/wheel.dae
- link sensor_frame: geometry collision mesh filename=../meshes/sensor_frame.stl scale=0.01 0.01 0.01; visual mesh filename=../meshes/sensor_frame.dae scale=0.01 0.01 0.01
- link top_chassis_link: geometry visual mesh filename=../meshes/top_chassis.dae
- link top_plate_link: geometry collision mesh filename=../meshes/top_plate.stl; visual mesh filename=../meshes/top_plate.dae
- link user_rail_link: geometry visual mesh filename=../meshes/user_rail.dae
